File: Board/AgitPOV_WiFi.sch (EAGLE design)
At the start: 41 parts, among them U1 MMA8452Q

Commit message: Cambios desde Manizales y Cartagena
- luz de colores en la pagina html
- individual AP desde el MAC address
Parts:
- removed JP-GND: SWITCH, SparkFun-Connectors:M01PTH
- removed JP1: (no value), SparkFun-Connectors:M01PTH
- added JPGND: switch, SparkFun-Connectors:M01PTH
- JP-GNDE: value - -> (none)
Connections:
- new net N$41: WEMOS2.3
- net GND: now also JPGND.1; no longer JP-GND.1
Other:
- moved on the sheet: JP-GNDE
Changed lines of the file:
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@@
 <part name="C1" library="SparkFun-Capacitors" deviceset="10UF-16V-10%(TANT)" device="" value="0.1uF"/>
 <part name="JST" library="con-garry" deviceset="332-02" device=""/>
-<part name="JP-GND" library="SparkFun-Connectors" deviceset="M01" device="PTH" value="SWITCH"/>
-<part name="JP-GNDE" library="SparkFun-Connectors" deviceset="M01" device="PTH" value="-"/>
 <part name="C2" library="SparkFun-Capacitors" deviceset="10UF-16V-10%(TANT)" device="" value="0.1uF"/>
 <part name="U1" library="SparkFun-Sensors" deviceset="MMA8452Q" device=""/>
 <part name="C3" library="SparkFun-Capacitors" deviceset="10UF-16V-10%(TANT)" device="" value="4.7uF"/>
-<part name="JP1" library="SparkFun-Connectors" deviceset="M01" device="PTH"/>
+<part name="JPGND" library="SparkFun-Connectors" deviceset="M01" device="PTH" value="switch"/>
+<part name="JP-GNDE" library="SparkFun-Connectors" deviceset="M01" device="PTH"/>
 </parts>
 <sheets>
@@
 <attribute name="NAME" x="61.722" y="25.4" size="1.524" layer="95" rot="R90"/>
 </instance>
-<instance part="JP-GND" gate="G$1" x="20.32" y="35.56" rot="MR180"/>
-<instance part="JP-GNDE" gate="G$1" x="81.28" y="20.32" rot="R180"/>
 <instance part="C2" gate="G$1" x="101.6" y="48.26"/>
 <instance part="U1" gate="G$1" x="127" y="50.8"/>
 <instance part="C3" gate="G$1" x="81.28" y="48.26"/>
-<instance part="JP1" gate="G$1" x="233.68" y="43.18"/>
+<instance part="JPGND" gate="G$1" x="20.32" y="33.02"/>
+<instance part="JP-GNDE" gate="G$1" x="81.28" y="22.86" rot="R180"/>
 </instances>
 <busses>
@@
 <pinref part="DEL12" gate="G$1" pin="GND"/>
 <wire x1="256.54" y1="76.2" x2="279.4" y2="76.2" width="0.1524" layer="91"/>
-<wire x1="27.94" y1="76.2" x2="27.94" y2="35.56" width="0.1524" layer="91"/>
+<wire x1="27.94" y1="76.2" x2="27.94" y2="33.02" width="0.1524" layer="91"/>
 <pinref part="WEMOS2" gate="G$1" pin="2"/>
 <wire x1="35.56" y1="35.56" x2="35.56" y2="43.18" width="0.1524" layer="91"/>
-<pinref part="JP-GND" gate="G$1" pin="1"/>
-<wire x1="27.94" y1="35.56" x2="35.56" y2="35.56" width="0.1524" layer="91"/>
-<wire x1="27.94" y1="35.56" x2="81.28" y2="35.56" width="0.1524" layer="91"/>
+<wire x1="27.94" y1="33.02" x2="35.56" y2="35.56" width="0.1524" layer="91"/>
+<wire x1="27.94" y1="33.02" x2="81.28" y2="35.56" width="0.1524" layer="91"/>
 <wire x1="81.28" y1="35.56" x2="81.28" y2="40.64" width="0.1524" layer="91"/>
 <wire x1="81.28" y1="40.64" x2="81.28" y2="43.18" width="0.1524" layer="91"/>
@@
 <wire x1="111.76" y1="43.18" x2="111.76" y2="40.64" width="0.1524" layer="91"/>
 <wire x1="116.84" y1="43.18" x2="111.76" y2="43.18" width="0.1524" layer="91"/>
+<pinref part="JPGND" gate="G$1" pin="1"/>
+<junction x="27.94" y="33.02"/>
 </segment>
 <segment>
@@
 <pinref part="JST" gate="-1" pin="S"/>
 <pinref part="BATT" gate="G$1" pin="1"/>
-<junction x="73.66" y="20.32"/>
 <pinref part="BATT" gate="G$1" pin="1"/>
-<wire x1="73.66" y1="20.32" x2="73.66" y2="10.16" width="0.1524" layer="91"/>
+<wire x1="73.66" y1="22.86" x2="73.66" y2="10.16" width="0.1524" layer="91"/>
 <junction x="73.66" y="10.16"/>
-<pinref part="JP-GNDE" gate="G$1" pin="1"/>
-<wire x1="73.66" y1="20.32" x2="60.96" y2="15.24" width="0.1524" layer="91"/>
+<wire x1="73.66" y1="22.86" x2="60.96" y2="15.24" width="0.1524" layer="91"/>
 <junction x="60.96" y="15.24"/>
 <wire x1="73.66" y1="10.16" x2="71.12" y2="10.16" width="0.1524" layer="91"/>
+<pinref part="JP-GNDE" gate="G$1" pin="1"/>
+<junction x="73.66" y="22.86"/>
 </segment>
 </net>
@@
 </segment>
 </net>
+<net name="N$41" class="0">
+<segment>
+<wire x1="38.1" y1="45.72" x2="38.1" y2="43.18" width="0.1524" layer="91"/>
+<pinref part="WEMOS2" gate="G$1" pin="3"/>
+</segment>
+</net>
